Commit message: rep

File: src/bot_demo/urdf/base.urdf.xacro (robot description, xacro)
@@ -50,12 +50,12 @@
     </gazebo>
     <joint name="caster_wheel_joint" type="fixed">
-        <parent link="base_link"/>
+        <parent link="chassis"/>
         <child link="caster_wheel"/>
-        <origin xyz="0.35 0 0" rpy="0 0 0"/>
+        <origin xyz="0.555 0 -0.05" rpy="0 0 0"/>
     </joint>
     <link name="caster_wheel">
         <visual>
             <geometry>
-                <sphere radius="0.074" />
+                <sphere radius="0.06" />
             </geometry>
             <material name="black"/>
@@ -63,8 +63,8 @@
         <collision>
             <geometry>
-                <sphere radius="0.074"/>
+                <sphere radius="0.06"/>
             </geometry>
         </collision>
-        <xacro:inertial_sphere mass="0.5"  radius="0.074">
+        <xacro:inertial_sphere mass="0.5"  radius="0.06">
             <origin xyz="0 0 0" rpy="0 0 0"/>
         </xacro:inertial_sphere>
@@ -78,5 +78,5 @@
         <parent link="base_link" />
         <child link="left_wheel" />
-        <origin xyz="0.0 0.2675 0.0" rpy="-1.5708 0 0"/>
+        <origin xyz="0.0 0.2775 -0.045" rpy="-1.5708 0 0"/>
         <axis xyz="0 0 1"/>
     </joint>
@@ -85,5 +85,5 @@
             <origin rpy="0 0 0" xyz="0 0 0" />
             <geometry>
-                <cylinder radius="0.074" length="0.043"/>
+                <cylinder radius="0.045" length="0.04"/>
             </geometry>
             <material name="Blue"/>
@@ -92,8 +92,8 @@
             <origin rpy="0 0 0" xyz="0 0 0" />
             <geometry>
-                <cylinder radius="0.074" length="0.043"/>
+                <cylinder radius="0.045" length="0.04"/>
             </geometry>
         </collision>
-        <xacro:inertial_cylinder mass="0.5" length="0.043" radius="0.074">
+        <xacro:inertial_cylinder mass="0.5" length="0.04" radius="0.09">
             <origin xyz="0 0 0" rpy="0 0 0"/>
         </xacro:inertial_cylinder>
@@ -105,5 +105,5 @@
         <parent link="base_link" />
         <child link="right_wheel" />
-        <origin xyz="0.0 -0.2675 0.0" rpy="1.5708 0 0"/>
+        <origin xyz="0.0 -0.2775 -0.045" rpy="1.5708 0 0"/>
         <axis xyz="0 0 -1"/>
     </joint>
@@ -112,5 +112,5 @@
             <origin rpy="0 0 0" xyz="0 0 0" />
             <geometry>
-                <cylinder radius="0.074" length="0.043"/>
+                <cylinder radius="0.045" length="0.04"/>
             </geometry>
             <material name="Blue"/>

File: src/bot_demo/urdf/robot.urdf.xacro (robot description, xacro)
@@ -3,5 +3,4 @@
     <xacro:include filename="base.urdf.xacro" />
     <xacro:include filename="laser.urdf.xacro" />
-    <xacro:include filename="camera.urdf.xacro" />
     <xacro:include filename="gazebo_control.xacro"/>
     <xacro:include filename="inertial_macros.xacro" />

Commit message: move_base change

File: src/bot_demo/urdf/base.urdf.xacro (robot description, xacro)
@@ -30,14 +30,14 @@
     <link name="chassis">
         <visual>
-            <origin xyz="0.3 0 0.15"/>
+            <origin xyz="0.3 0 0.125"/>
             <geometry>
-                <box size="0.6 0.485 0.3"/>
+                <box size="0.6 0.485 0.25"/>
             </geometry>
             <material name="White"/>
         </visual>
         <collision>
-            <origin xyz="0.3 0 0.15"/>
+            <origin xyz="0.3 0 0.125"/>
             <geometry>
-                <box size="0.6 0.485 0.3"/>
+                <box size="0.6 0.485 0.25"/>
             </geometry>
         </collision>
@@ -52,5 +52,5 @@
         <parent link="chassis"/>
         <child link="caster_wheel"/>
-        <origin xyz="0.555 0 -0.05" rpy="0 0 0"/>
+        <origin xyz="0.555 0 -0.014" rpy="0 0 0"/>
     </joint>
     <link name="caster_wheel">
@@ -78,5 +78,5 @@
         <parent link="base_link" />
         <child link="left_wheel" />
-        <origin xyz="0.0 0.2775 -0.045" rpy="-1.5708 0 0"/>
+        <origin xyz="0.0 0.2775 -0.029" rpy="-1.5708 0 0"/>
         <axis xyz="0 0 1"/>
     </joint>
@@ -105,5 +105,5 @@
         <parent link="base_link" />
         <child link="right_wheel" />
-        <origin xyz="0.0 -0.2775 -0.045" rpy="1.5708 0 0"/>
+        <origin xyz="0.0 -0.2775 -0.029" rpy="1.5708 0 0"/>
         <axis xyz="0 0 -1"/>
     </joint>
@@ -129,26 +129,3 @@
         <material>Gazebo/Blue</material>
     </gazebo>
-   <!--<joint name="laser_joint" type="fixed">
-        <origin xyz="0.555 0 0.325" rpy="0 0 0" />
-        <parent link="chassis" />
-        <child link="laser" />
-    </joint>
-    <link name="laser">
-        <visual>
-        <origin rpy="0 0 -1.5708" xyz="0 0 0"/>
-        <geometry>
-            <mesh filename="package://bot_demo/stl/rplidar.stl" scale="0.001 0.001 0.001"/>
-        </geometry>
-        <material name="Yellow"/>
-        </visual>
-        <collision>
-        <origin rpy="0 0 0" xyz="0 0 0"/>
-        <geometry>
-            <mesh filename="package://bot_demo/stl/rplidar.stl" scale="0.001 0.001 0.001"/>
-        </geometry>
-        </collision>
-    </link>
-    <gazebo reference="laser">
-        <material>Gazebo/Yellow</material>
-    </gazebo>-->
 </robot>

File: src/bot_demo/urdf/laser.urdf.xacro (robot description, xacro)
@@ -19,5 +19,5 @@
     </gazebo>
     <joint name="laser_joint" type="fixed">
-        <origin xyz="0.555 0 0.325" rpy="0 0 0" />
+        <origin xyz="0.555 0 0.275" rpy="0 0 0" />
         <parent link="chassis" />
         <child link="laser" />

Commit message: change

File: src/bot_demo/urdf/base.urdf.xacro (robot description, xacro)
@@ -43,5 +43,5 @@
         </collision>
         <xacro:inertial_box mass="5.0" x="0.6" y="0.485" z="0.25">
-            <origin xyz="0.3 0 0.15" rpy="0 0 0"/>
+            <origin xyz="0.3 0 0.125" rpy="0 0 0"/>
         </xacro:inertial_box>
     </link>
@@ -95,5 +95,5 @@
             </geometry>
         </collision>
-        <xacro:inertial_cylinder mass="0.5" length="0.04" radius="0.09">
+        <xacro:inertial_cylinder mass="0.5" length="0.04" radius="0.045">
             <origin xyz="0 0 0" rpy="0 0 0"/>
         </xacro:inertial_cylinder>
@@ -119,8 +119,8 @@
             <origin rpy="0 0 0" xyz="0 0 0" />
             <geometry>
-                <cylinder radius="0.074" length="0.043"/>
+                <cylinder radius="0.045" length="0.04"/>
             </geometry>
         </collision>
-        <xacro:inertial_cylinder mass="0.5" length="0.043" radius="0.074">
+        <xacro:inertial_cylinder mass="0.5" length="0.04" radius="0.045">
             <origin xyz="0 0 0" rpy="0 0 0"/>
         </xacro:inertial_cylinder>

File: src/bot_demo/urdf/robot.urdf.xacro (robot description, xacro)
@@ -3,6 +3,6 @@
     <xacro:include filename="base.urdf.xacro" />
     <xacro:include filename="laser.urdf.xacro" />
+    <xacro:include filename="gazebo_control.xacro" />
     <xacro:include filename="inertial_macros.xacro" />
-    <xacro:include filename="mycamera.urdf.xacro" />
     <xacro:include filename="mylaser.urdf.xacro" />
 </robot>

Commit message: Update base.urdf.xacro

File: src/bot_demo/urdf/base.urdf.xacro (robot description, xacro)
@@ -18,4 +18,11 @@
     <link name="base_link">
     </link>
+    <link name="imu_link">
+    </link>
+    <joint name="imu_joint" type="fixed">
+        <parent link="base_link"/>
+        <child link="imu_link"/>
+        <origin xyz="0 0 0.05" rpy="0 0 0"/>
+    </joint>
     <joint name="base_footprint_joint" type="fixed">
         <parent link="base_footprint"/>
@@ -26,5 +33,5 @@
         <parent link="base_link"/>
         <child link="chassis"/>
-        <origin xyz="-0.1 0 0"/>
+        <origin xyz="-0.06 0 0"/>
     </joint>
     <link name="chassis">
@@ -129,3 +136,46 @@
         <material>Gazebo/Blue</material>
     </gazebo>
+    <link name="camera_link">
+    </link>
+    <joint name="camera_to_base_joint" type="fixed">
+        <parent link="base_link"/>
+        <child link="camera_link"/>
+        <origin xyz="0.24 0 0.62" rpy="0 0 0"/>
+    </joint>
+    <link name="camera_color_frame"/>
+    <link name="camera_color_optical_frame"/>
+    <joint name="camera_color_joint" type="fixed">
+        <parent link="camera_link"/>
+        <child link="camera_color_frame"/>
+        <origin xyz="0 0 0" rpy="0 0 0"/>
+    </joint>
+    <joint name="camera_color_optical_joint" type="fixed">
+        <parent link="camera_color_frame"/>
+        <child link="camera_color_optical_frame"/>
+        <origin xyz="0 0 0" rpy="-1.5708 0 -1.5708"/>
+    </joint>
+    <link name="camera_depth_frame"/>
+    <link name="camera_depth_optical_frame"/>
+    <joint name="camera_depth_joint" type="fixed">
+        <parent link="camera_link"/>
+        <child link="camera_depth_frame"/>
+        <origin xyz="0 0 0" rpy="0 0 0"/>
+    </joint>
+    <joint name="camera_depth_optical_joint" type="fixed">
+        <parent link="camera_depth_frame"/>
+        <child link="camera_depth_optical_frame"/>
+        <origin xyz="0 0 0" rpy="-1.5708 0 -1.5708"/>
+    </joint>
+    <link name="camera_ir_frame"/>
+    <link name="camera_ir_optical_frame"/>
+    <joint name="camera_ir_joint" type="fixed">
+        <parent link="camera_link"/>
+        <child link="camera_ir_frame"/>
+        <origin xyz="0 0 0" rpy="0 0 0"/>
+    </joint>
+    <joint name="camera_ir_optical_joint" type="fixed">
+        <parent link="camera_ir_frame"/>
+        <child link="camera_ir_optical_frame"/>
+        <origin xyz="0 0 0" rpy="-1.5708 0 -1.5708"/>
+    </joint>
 </robot>
